Commit message: final commit

File: software Whole-body Motion Planning and Control for underactuated  wheeled-bipedal robots/robot.urdf (robot description, URDF)
Before this commit: robot tita, 15 links, 14 joints
Links:
- added link base_r_link
- added link base_t_link
- added link base_x_link
- added link base_y_link
- added link base_z_link
- added link world_origin
- link base_link: geometry collision box size=0.47 0.3 0.19; visual mesh filename=meshes/base_link.STL
- link left_leg_1: geometry visual mesh filename=meshes/left_leg_1.STL
- link left_leg_2: geometry visual mesh filename=meshes/left_leg_2.STL
- link left_leg_3: geometry collision box size=0.2 0.07 0.05; visual mesh filename=meshes/left_leg_3.STL
- link left_leg_4: geometry collision cylinder length=0.034 radius=0.0925; visual mesh filename=meshes/left_leg_4.STL
- link right_leg_1: geometry visual mesh filename=meshes/right_leg_1.STL
- link right_leg_2: geometry visual mesh filename=meshes/right_leg_2.STL
- link right_leg_3: geometry collision box size=0.2 0.07 0.05; visual mesh filename=meshes/right_leg_3.STL
- link right_leg_4: geometry collision cylinder length=0.034 radius=0.0925; visual mesh filename=meshes/right_leg_4.STL
Joints:
- added joint base_pitch_joint: type continuous, parent base_t_link, child base_link, origin xyz=0 0 0 rpy=0 0 0, axis 0 1 0
- added joint base_roll_joint: type continuous, parent base_r_link, child base_t_link, origin xyz=0 0 0 rpy=0 0 0, axis 1 0 0
- added joint base_x_joint: type prismatic, parent world_origin, child base_x_link, origin xyz=0 0 0 rpy=0 0 0, axis 1 0 0, limit lower=-100 upper=100 effort=100.0 velocity=100.0
- added joint base_y_joint: type prismatic, parent base_x_link, child base_y_link, origin xyz=0 0 0 rpy=0 0 0, axis 0 1 0, limit lower=-100 upper=100 effort=100.0 velocity=100.0
- added joint base_yaw_joint: type continuous, parent base_z_link, child base_r_link, origin xyz=0 0 0 rpy=0 0 0, axis 0 0 1
- added joint base_z_joint: type prismatic, parent base_y_link, child base_z_link, origin xyz=0 0 0 rpy=0 0 0, axis 0 0 1, limit lower=-100 upper=100 effort=100.0 velocity=100.0
